File: TL59025_devboard.kicad_pcb (KiCad board)
At the start: 2 copper layers, 61 x 41 mm, 67 parts, among them J1 UPDI, J2 USB_C_Receptacle_USB2.0, J3 Cascade In, J4 Cascade Out, SW1 SW_Push, U1 AMS1117-3.3, U2 ATtiny414-SS, U3 CH340E, U4 TL59025, U5 TL59025

Commit message: Change R3 and R4 to 510R for maximum current range
Parts:
- R3, R4: value 1K -> 510R
Changed lines of the file:
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@@
       (effects (font (size 1 1) (thickness 0.15)))
     )
-    (fp_text value "1K" (at 0 1.43 90) (layer "F.Fab")
+    (fp_text value "510R" (at 0 1.43 90) (layer "F.Fab")
       (effects (font (size 1 1) (thickness 0.15)))
     )
@@
       (effects (font (size 1 1) (thickness 0.15)))
     )
-    (fp_text value "1K" (at 0 1.43 90) (layer "F.Fab")
-      (effects (font (size 1 1) (thickness 0.15)))
-    )
+    (fp_text value "510R" (at 0 1.43 90) (layer "F.Fab")
+      (effects (font (size 1 1) (thickness 0.15)))
+    )
